Commit message: slam_toolbox

File: slambot_gazebo_sim_description/urdf/slambot_gazebo_sim.xacro (robot description, xacro)
@@ -175,5 +175,5 @@
   <dynamics damping="0.1" friction="0.0"/>
 </joint>
-<joint name="${prefix}Lidar_joint" type="continuous">
+<joint name="${prefix}Lidar_joint" type="fixed">
   <origin xyz="-0.0785 0.0 0.118031" rpy="0 0 0"/>
   <parent link="${prefix}base_link"/>

Commit message: good

File: slambot_gazebo_sim_description/urdf/slambot_gazebo_sim.xacro (robot description, xacro)
@@ -27,5 +27,5 @@
 <link name="${prefix}FL_wheel">
   <inertial>
-    <origin xyz="-6.938893903907228e-18 0.011499999776482576 -6.938893903907228e-18" rpy="0 0 0"/>
+    <origin xyz="0 0.0115 0" rpy="0 0 0"/>
     <mass value="0.075"/>
     <inertia ixx="2.4e-05" iyy="4.1e-05" izz="2.4e-05" ixy="0.0" iyz="0.0" ixz="0.0"/>
@@ -47,5 +47,5 @@
 <link name="${prefix}BL_wheel">
   <inertial>
-    <origin xyz="0.0 0.011499999776482604 -6.938893903907228e-18" rpy="0 0 0"/>
+    <origin xyz="0.0 0.0115 0" rpy="0 0 0"/>
     <mass value="0.075"/>
     <inertia ixx="2.4e-05" iyy="4.1e-05" izz="2.4e-05" ixy="0.0" iyz="-0.0" ixz="0.0"/>
@@ -67,5 +67,5 @@
 <link name="${prefix}FR_wheel">
   <inertial>
-    <origin xyz="6.938893903907228e-17 -0.011499999776482757 -1.700029006457271e-16" rpy="0 0 0"/>
+    <origin xyz="0 -0.0115 0" rpy="0 0 0"/>
     <mass value="0.075"/>
     <inertia ixx="2.4e-05" iyy="4.1e-05" izz="2.4e-05" ixy="-0.0" iyz="-0.0" ixz="0.0"/>
@@ -87,5 +87,5 @@
 <link name="${prefix}BR_wheel">
   <inertial>
-    <origin xyz="-2.3681641159872813e-07 -0.011499999776482618 3.469446951953614e-18" rpy="0 0 0"/>
+    <origin xyz="0 -0.0115 0" rpy="0 0 0"/>
     <mass value="0.075"/>
     <inertia ixx="2.4e-05" iyy="4.1e-05" izz="2.4e-05" ixy="-0.0" iyz="0.0" ixz="0.0"/>
@@ -107,6 +107,6 @@
 <link name="${prefix}Lidar">
   <inertial>
-    <origin xyz="0.0 0.0 0.029000013286372167" rpy="0 0 0"/>
-    <mass value="1.7521997405948053"/>
+    <origin xyz="0.0 0.0 0.029" rpy="0 0 0"/>
+    <mass value="1.0"/>
     <inertia ixx="0.001028" iyy="0.001028" izz="0.001073" ixy="0.0" iyz="0.0" ixz="0.0"/>
   </inertial>

Commit message: 소프트 네비 완성본

File: slambot_gazebo_sim_description/urdf/slambot_gazebo_sim.xacro (robot description, xacro)
@@ -5,4 +5,5 @@
 <xacro:include filename="$(find slambot_gazebo_sim_description)/urdf/slambot_gazebo_sim.trans" />
 <xacro:include filename="$(find slambot_gazebo_sim_description)/urdf/slambot_gazebo_sim.gazebo" />
+<xacro:property name="wheel_radius" value="0.031"/>
 <link name="${prefix}base_link">
   <inertial>
@@ -148,5 +149,5 @@
 </link>
 <joint name="${prefix}FL_joint" type="continuous">
-  <origin xyz="0.058 0.05705 0.0221" rpy="0 0 0"/>
+  <origin xyz="0.058 0.05705 ${wheel_radius}" rpy="0 0 0"/>
   <parent link="${prefix}base_link"/>
   <child link="${prefix}FL_wheel"/>
@@ -155,5 +156,5 @@
 </joint>
 <joint name="${prefix}BL_joint" type="continuous">
-  <origin xyz="-0.055 0.05705 0.0221" rpy="0 0 0"/>
+  <origin xyz="-0.055 0.05705 ${wheel_radius}" rpy="0 0 0"/>
   <parent link="${prefix}base_link"/>
   <child link="${prefix}BL_wheel"/>
@@ -162,5 +163,5 @@
 </joint>
 <joint name="${prefix}FR_joint" type="continuous">
-  <origin xyz="0.058 -0.05705 0.0221" rpy="0 0 0"/>
+  <origin xyz="0.058 -0.05705 ${wheel_radius}" rpy="0 0 0"/>
   <parent link="${prefix}base_link"/>
   <child link="${prefix}FR_wheel"/>
@@ -169,5 +170,5 @@
 </joint>
 <joint name="${prefix}BR_joint" type="continuous">
-  <origin xyz="-0.055 -0.05705 0.0221" rpy="0 0 0"/>
+  <origin xyz="-0.055 -0.05705 ${wheel_radius}" rpy="0 0 0"/>
   <parent link="${prefix}base_link"/>
   <child link="${prefix}BR_wheel"/>
